File: examples/layout/ato/pcb.kicad_pcb (KiCad board)
At the start: 2 copper layers, 2 parts

Commit message: Picker: Remove sqlite picker (#665)
Extra:
- Disable cachepicker (performance)
- Fix battery pick
Parts:
- R1: value 10kΩ ±1% 62.5mW -> 8.2kΩ ±1% 62.5mW
Changed lines of the file:
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@@
                     (thickness 0.15))
                 (hide no)))
-        (property "Value" "10kΩ ±1% 62.5mW"
+        (property "Value" "8.2kΩ ±1% 62.5mW"
             (at 0 4 0)
             (layer "F.Fab")
@@
                     (thickness 0.15))
                 (hide yes)))
-        (property "LCSC" "C25744"
+        (property "LCSC" "C25924"
             (at 0 0 0)
             (layer "User.9")

Commit message: Deps: Remove networkx, igraph; Remove routing (#710)
Remove networkx and igraph dep by removing routing
Parts:
- removed C1: 100nF ±10% 16V X7R, lcsc:C0402
- removed R1: 8.2kΩ ±1% 62.5mW, lcsc:R0402
