File: examples/layout/power_logger/power_logger.kicad_pcb (KiCad board)
At the start: 2 copper layers, 50 x 66 mm, 51 parts

Commit message: add access_control example
Parts:
- R6: value 0Ω 250mW -> 25mΩ ±1% 1W; footprint UNI_ROYAL_1206W4F0000T5E:R1206 -> jieerrui_JER1206F1R025:R1206
Connections:
- Card1 pad 3: line-1 -> line-9
- Card1 pad 5: line -> line-5
- Card1 pad 7: line-2 -> line-4
- R11 pad 1: line-5 -> line-2
- R14 pad 1: line-3 -> line
- R15 pad 1: line-4 -> line-1
- R4 pad 1: input-2 -> input-1
- R5 pad 1: input-1 -> input-2
- SW1 pad 1: input-2 -> input-1
- SW1 pad 2: output-2 -> output-1
- SW2 pad 1: input-1 -> input-2
- SW2 pad 2: output-1 -> output-2
- U1 pad 3: line-6 -> line-3
- U2 pad 7: A0 -> gnd-1
- U4 pad 12: line-3 -> line
- U4 pad 13: line-4 -> line-1
- U4 pad 18: line-2 -> line-4
- U4 pad 19: line -> line-5
- U4 pad 20: line-1 -> line-9
- U4 pad 21: output-1 -> output-2
- U4 pad 26: line-7 -> line-6
- U4 pad 27: line-8 -> line-7
- U4 pad 30: line-9 -> line-8
- U4 pad 31: output-2 -> output-1
- U4 pad 5: line-5 -> line-2
- U4 pad 6: line-6 -> line-3
- U6 pad 2: line-4 -> line-1
- U6 pad 3: line-3 -> line
- USB1 pad A6: line-8 -> line-7
- USB1 pad A7: line-7 -> line-6
- USB1 pad B6: line-8 -> line-7
- USB1 pad B7: line-7 -> line-6
Routing:
- net line-3: track 15.8 -> 38.0 mm, vias 0 -> 4
- net output-2: track 5.41 -> 26.6 mm, vias 0 -> 2
- net output-1: track 26.6 -> 5.41 mm, vias 2 -> 0
- net line-6: track 38.0 -> 17.5 mm, vias 4 -> 2
- net line-9: track 0.00 -> 20.0 mm
- net line-2: track 21.2 -> 1.47 mm
- net line-5: track 1.47 -> 20.6 mm
- net line-8: track 18.1 -> 0.00 mm, vias 2 -> 0
- net line: track 20.6 -> 15.8 mm
- net line-4: track 17.0 -> 21.2 mm
- net line-1: track 20.0 -> 17.0 mm
- net input-2: track 1.14 -> 1.86 mm
- net input-1: track 1.86 -> 1.14 mm
- net line-7: track 17.5 -> 18.1 mm
