File: examples/led_badge/layouts/strip10/strip10.kicad_pcb (KiCad board)
At the start: 2 copper layers, 20 parts

Commit message: just need usb to work
Connections:
- net -DOUT-0 renamed DOUT
- net -DOUT-1 renamed leds[1]-data_in-DIN
- net -DOUT-2 renamed leds[2]-data_in-DIN
- net -DOUT-3 renamed leds[3]-data_in-DIN
- net -DOUT-4 renamed leds[4]-data_in-DIN
- net -DOUT-5 renamed leds[5]-data_in-DIN
- net -DOUT-6 renamed leds[6]-data_in-DIN
- net -DOUT-7 renamed leds[7]-data_in-DIN
- net -DOUT-8 renamed leds[8]-data_in-DIN
- net -DOUT-9 renamed leds[9]-data_in-DIN
- net DIN renamed leds[0]-data_in-DIN
- net gnd renamed GND
- net hv renamed VCC
