File: test/common/resources/fileformats/kicad/v9/pcb/test.kicad_pcb (KiCad board)
At the start: 2 copper layers, 4 parts

Commit message: Exporters: KiCad file format: Add support for custom fonts (#1453)
## Description

Add basic support for custom fonts in text objects in the kivas file
format.
No font embedding yet.

## Motivation

Every build would delete all custom fonts and setting in the PCB design.
Other:
- board text added: "TEST_B"
Changed lines of the file:
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@@
+		)
+	)
+	(gr_text "TEST_B"
+		(at 34 31.5 315)
+		(layer "B.SilkS")
+		(effects
+			(font
+				(size 1 1)
+				(thickness 0.1)
+				(italic yes)
+			)
+			(justify mirror)
+		)
+	)
+	(gr_text_box "TEST"
+		(pts
+			(xy 27 17) (xy 34.071068 9.928932) (xy 39.374369 15.232233) (xy 32.303301 22.303301)
+		)
+		(margins 1.0025 1.0025 1.0025 1.0025)
+		(angle 45)
+		(layer "F.SilkS")
+		(effects
+			(font
+				(size 1 1)
+				(thickness 0.2)
+				(bold yes)
+				(italic yes)
+			)
+			(justify left top)
+		)
+		(border yes)
+		(stroke
+			(width 0.1)
+			(type solid)
+		)
+	)
+	(gr_text_box "TEST"
+		(start 23.187184 12.366117)
+		(end 33.187184 19.866117)
+		(margins 1.0025 1.0025 1.0025 1.0025)
+		(layer "F.SilkS")
+		(effects
+			(font
+				(size 1 1)
+				(thickness 0.125)
+			)
+			(justify right bottom)
+		)
+		(border yes)
+		(stroke
+			(width 0.1)
+			(type solid)
 		)
 	)
