File: test/common/resources/fileformats/kicad/v9/pcb/test.kicad_pcb (KiCad board)
At the start: 2 copper layers, 4 parts

Commit message: add testcase to test file
Other:
- board text added: "Multi-line text newline return single backslash \ double backslash \\ tab> <tab"
Changed lines of the file:
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@@
 			(usegerberadvancedattributes yes)
 			(creategerberjobfile yes)
-			(dashed_line_dash_ratio 12)
-			(dashed_line_gap_ratio 3)
+			(dashed_line_dash_ratio 12.000000)
+			(dashed_line_gap_ratio 3.000000)
 			(svgprecision 4)
 			(plotframeref no)
@@
 			(hpglpennumber 1)
 			(hpglpenspeed 20)
-			(hpglpendiameter 15)
+			(hpglpendiameter 15.000000)
 			(pdf_front_fp_property_popups yes)
 			(pdf_back_fp_property_popups yes)
@@
 			)
 		)
+	)
+	(gr_text "Multi-line text\nnewline\nreturn\nsingle backslash \\\ndouble backslash \\\\\ntab>	<tab"
+		(at 26.5 31.5 0)
+		(layer "F.SilkS")
+		(effects
+			(font
+				(size 0.5 0.5)
+				(thickness 0.1)
+			)
+		)

Commit message: fix tab parsing (kicad can read double-char-tab and literal-tab, but dumps only literal tab)
Other:
- board text added: "Multi-line text newline returnr single backslash \ double backslash \\ tab> <tab"
- board text removed: "Multi-line text newline return single backslash \ double backslash \\ tab> <tab"
Changed lines of the file:
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@@
 			(usegerberadvancedattributes yes)
 			(creategerberjobfile yes)
-			(dashed_line_dash_ratio 12.000000)
-			(dashed_line_gap_ratio 3.000000)
+			(dashed_line_dash_ratio 12)
+			(dashed_line_gap_ratio 3)
 			(svgprecision 4)
 			(plotframeref no)
@@
 			(hpglpennumber 1)
 			(hpglpenspeed 20)
-			(hpglpendiameter 15.000000)
+			(hpglpendiameter 15)
 			(pdf_front_fp_property_popups yes)
 			(pdf_back_fp_property_popups yes)
@@
 		)
 	)
-	(gr_text "Multi-line text\nnewline\nreturn\nsingle backslash \\\ndouble backslash \\\\\ntab>	<tab"
+	(gr_text "Multi-line text\nnewline\nreturn\r\nsingle backslash \\\ndouble backslash \\\\\ntab>	<tab"
 		(at 26.5 31.5 0)
 		(layer "F.SilkS")
