File: examples/led_badge/layouts/badge/badge.kicad_pcb (KiCad board)
At the start: 4 copper layers, 56.3 x 39 mm, 240 parts

Commit message: layout tidy
Parts:
- moved L1 0.20 mm to (114.9, 109.2)
Routing:
- net power_system: track 25.9 -> 16.3 mm, vias 4 -> 3
- net power_battery: track 27.9 -> 30.6 mm, vias 2 -> 4
- net gnd: vias 216 -> 215
- net (no net): vias 2 -> 0
