File: examples/layout_reuse/layout/sub/sub.kicad_pcb (KiCad board)
At the start: 2 copper layers, 3 parts

Commit message: pr-cleanup: drop unrelated examples changes
Parts:
- R1, R2, R3: value 1000Ω -> 1kΩ
Changed lines of the file:
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@@
 	)
 	(setup
-		(stackup
-			(layer "F.SilkS"
-				(type "Top Silk Screen")
-			)
-			(layer "F.Paste"
-				(type "Top Solder Paste")
-			)
-			(layer "F.Mask"
-				(type "Top Solder Mask")
-				(color "Black")
-				(thickness 0.01)
-				(material "Solder mask")
-				(epsilon_r 3.3)
-			)
-			(layer "F.Cu"
-				(type "copper")
-				(thickness 0.035)
-			)
-			(layer "dielectric 1"
-				(type "core")
-				(thickness 1.51)
-				(material "FR4")
-				(epsilon_r 4.5)
-				(loss_tangent 0.02)
-			)
-			(layer "B.Cu"
-				(type "copper")
-				(thickness 0.035)
-			)
-			(layer "B.Mask"
-				(type "Bottom Solder Mask")
-				(color "Black")
-				(thickness 0.01)
-				(material "Solder mask")
-				(epsilon_r 3.3)
-			)
-			(layer "B.Paste"
-				(type "Bottom Solder Paste")
-			)
-			(layer "B.SilkS"
-				(type "Bottom Silk Screen")
-			)
-			(copper_finish "ENIG")
-		)
 		(pad_to_mask_clearance 0)
 		(allow_soldermask_bridges_in_footprints no)
@@
 			)
 		)
-		(property "Value" "1000Ω"
+		(property "Value" "1kΩ"
 			(at 0 4)
 			(layer "F.Fab")
@@
 			(hide yes)
 		)
-		(property "resistance" "1000±1.0%Ω"
-			(at 0 0 0)
-			(layer "User.9")
-			(hide yes)
-		)
-		(property "max_power" "0.062W"
-			(at 0 0 0)
-			(layer "User.9")
-			(hide yes)
-		)
-		(property "max_voltage" "50V"
+		(property "resistance" "1±20.0%kΩ"
+			(at 0 0 0)
+			(layer "User.9")
+			(hide yes)
+		)
+		(property "max_power" "any ≥0W"
+			(at 0 0 0)
+			(layer "User.9")
+			(hide yes)
+		)
+		(property "max_voltage" "any ≥0V"
 			(at 0 0 0)
 			(layer "User.9")
@@
 			)
 		)
-		(property "Value" "1000Ω"
+		(property "Value" "1kΩ"
 			(at 0 4)
 			(layer "F.Fab")
@@
 			(hide yes)
 		)
-		(property "resistance" "1000±1.0%Ω"
-			(at 0 0 0)
-			(layer "User.9")
-			(hide yes)
-		)
-		(property "max_power" "0.062W"
-			(at 0 0 0)
-			(layer "User.9")
-			(hide yes)
-		)
-		(property "max_voltage" "50V"
+		(property "resistance" "1±20.0%kΩ"
+			(at 0 0 0)
+			(layer "User.9")
+			(hide yes)
+		)
+		(property "max_power" "any ≥0W"
+			(at 0 0 0)
+			(layer "User.9")
+			(hide yes)
+		)
+		(property "max_voltage" "any ≥0V"
 			(at 0 0 0)
 			(layer "User.9")
@@
 			)
 		)
-		(property "Value" "1000Ω"
+		(property "Value" "1kΩ"
 			(at 0 4)
 			(layer "F.Fab")
@@
 			(hide yes)
 		)
-		(property "resistance" "1000±1.0%Ω"
-			(at 0 0 0)
-			(layer "User.9")
-			(hide yes)
-		)
-		(property "max_power" "0.062W"
-			(at 0 0 0)
-			(layer "User.9")
-			(hide yes)
-		)
-		(property "max_voltage" "50V"
-			(at 0 0 0)
-			(layer "User.9")
+		(property "resistance" "1±20.0%kΩ"
+			(at 0 0 0)
+			(layer "User.9")
+			(hide yes)
+		)
+		(property "max_power" "any ≥0W"
+			(at 0 0 0)
+			(layer "User.9")
+			(hide yes)
+		)
+		(property "max_voltage" "any ≥0V"
+			(at 0 0 0)
+			(layer "User.9")
