File: test/common/resources/fileformats/kicad/v8/pcb/test.kicad_pcb (KiCad board)
At the start: 2 copper layers, 4 parts

Commit message: agent: remove duplicate path tool aliases
Parts:
- G***: moved to B.Cu
- turned G*** to 180 degrees
