File: examples/buck_converter/layouts/simulation/simulation.kicad_pcb (KiCad board)
At the start: 2 copper layers, 14 parts

Commit message: final checkin
Parts:
- removed C5: 0F, Chinocera_HGC1210R5107M160NSVK:C1210
- added R7: 91000Ω, YAGEO_RC0402FR_0791KL:R0402, F.Cu at (0.00, 0.00)
- C2: footprint YAGEO_CC0603JRNPO9BN8R2:C0603 -> Samsung_Electro_Mechanics_CL10C470JB8NNNC:C0603
- C3: footprint FH_0805B333K500NT:C0805 -> FH_0805B472K500NT:C0805
- L1: footprint Sunlord_SWPA8040S2R2MT:IND-SMD_L8.0-W8.0_SWPA8040S -> YJYCOIN_YNR8040_6R8M:IND-SMD_L8.0-W8.0
- R1: value 7680Ω -> 10200Ω; footprint UNI_ROYAL_0402WGF7681TCE:R0402 -> UNI_ROYAL_0402WGF1022TCE:R0402
- R2: value 23700Ω -> 16900Ω; footprint YAGEO_RC0402FR_0723K7L:R0402 -> UNI_ROYAL_0402WGF1692TCE:R0402
- R3: value 100000Ω -> 450000Ω; footprint UNI_ROYAL_0402WGF1003TCE:R0402 -> FOJAN_FRC0402F4503TS:R0402
- R5: value 95300Ω -> 243000Ω; footprint Vishay_Intertech_CRCW040295K3FKED:R0402 -> UNI_ROYAL_0402WGF2433TCE:R0402
- R6: value 40200Ω -> 53600Ω; footprint UNI_ROYAL_0402WGF4022TCE:R0402 -> UNI_ROYAL_0402WGF5362TCE:R0402
Routing:
- net power_out-hv: track 26.8 -> 0.00 mm, vias 21 -> 0
- net 12: track 0.00 -> 26.8 mm, vias 0 -> 21
- net EN: track 2.06 -> 0.00 mm
- net 20: track 0.00 -> 2.06 mm

Commit message: checkin from server
Parts:
- R1: value 10200Ω -> 53600Ω; footprint UNI_ROYAL_0402WGF1022TCE:R0402 -> UNI_ROYAL_0402WGF5362TCE:R0402
- R3: value 450000Ω -> 91000Ω; footprint FOJAN_FRC0402F4503TS:R0402 -> YAGEO_RC0402FR_0791KL:R0402
- R4: value 1Ω -> 450000Ω; footprint UNI_ROYAL_1210W2F100KT5E:R1210 -> FOJAN_FRC0402F4503TS:R0402
- R5: value 243000Ω -> 1Ω; footprint UNI_ROYAL_0402WGF2433TCE:R0402 -> UNI_ROYAL_1210W2F100KT5E:R1210
- R6: value 53600Ω -> 240000Ω; footprint UNI_ROYAL_0402WGF5362TCE:R0402 -> FOJAN_FRC0402F2403TS:R0402
- R7: value 91000Ω -> 10000Ω; footprint YAGEO_RC0402FR_0791KL:R0402 -> UNI_ROYAL_0603WAF1002T5E:R0603
- moved R3 221.4 mm to (40.0, -200.0)
- moved R1 195.5 mm to (0.00, -10.0)
- moved R4 22.4 mm to (-142.0, -109.4)
- moved R6 22.4 mm to (-142.0, -119.4)
- moved C1 20.0 mm to (-142.0, -159.4)
- moved C2 20.0 mm to (-142.0, -139.4)
- moved C3 20.0 mm to (-142.0, -149.4)
- moved C4 20.0 mm to (-132.0, -109.4)
- moved D1 20.0 mm to (-142.0, -109.4)
- moved L1 20.0 mm to (11.9, -0.80)
- moved R2 20.0 mm to (-142.0, -129.4)
- moved R5 20.0 mm to (-142.0, -119.4)
- moved U1 20.0 mm to (20.0, 0.00)
Connections:
- L1 pad 1: (no net) -> cathode
- L1 pad 2: (no net) -> ref_in-hv
- R1 pad 1: FB -> ref_in-hv
- R1 pad 2: anode -> ref_out-hv
- R3 pad 1: power_in-hv -> EN
- R3 pad 2: EN -> anode
- R4 pad 1: power_out-hv -> power_in-hv
- R4 pad 2: anode -> EN
- R5 pad 1: RT_CLK -> ref_in-hv
- R6 pad 1: power_out-hv -> RT_CLK
- R6 pad 2: FB -> anode
- R7 pad 1: EN -> ref_out-hv
- U1 pad 5: FB -> ref_out-hv
Routing:
- net 0: track 32.8 -> 68.5 mm, vias 14 -> 35
- net 12: track 26.8 -> 0.00 mm, vias 21 -> 0
- net FB: track 9.00 -> 0.00 mm
- net EN: track 0.00 -> 2.06 mm
- net 20: track 2.06 -> 0.00 mm
- added copper zone on F.Cu, net c_in-power-hv
- removed copper zone on F.Cu, net output_caps[3]-power-hv
- removed copper zone on F.Cu, net power_out-hv
