File: examples/buck_converter/layouts/design-validation/design-validation.kicad_pcb (KiCad board)
At the start: 2 copper layers, 14 parts

Commit message: checkin from server
Parts:
- added C10: 0F, Samsung_Electro_Mechanics_CL10C470JB8NNNC:C0603, F.Cu at (60.0, -20.0)
- added C11: 0F, FH_0805B472K500NT:C0805, F.Cu at (60.0, -260.0)
- added C12: 0F, Samsung_Electro_Mechanics_CL21A106KAYNNNE:C0805, F.Cu at (60.0, -300.0)
- added C5: 0F, YAGEO_CC0603KRX7R9BB104:C0603, F.Cu at (60.0, -180.0)
- added C6: 0F, Samsung_Electro_Mechanics_CL10C470JB8NNNC:C0603, F.Cu at (60.0, -280.0)
- added C7: 0F, FH_0805B472K500NT:C0805, F.Cu at (60.0, -170.0)
- added C8: 0F, Samsung_Electro_Mechanics_CL21A106KAYNNNE:C0805, F.Cu at (60.0, -230.0)
- added C9: 0F, YAGEO_CC0603KRX7R9BB104:C0603, F.Cu at (60.0, -270.0)
- added D2: , STMicroelectronics_STPS340U:SMB_L4.6-W3.6-LS5.3-RD, F.Cu at (30.0, 0.00)
- added D3: , STMicroelectronics_STPS340U:SMB_L4.6-W3.6-LS5.3-RD, F.Cu at (50.0, 0.00)
- added L2: L 0H, YJYCOIN_YNR8040_6R8M:IND-SMD_L8.0-W8.0, F.Cu at (60.0, -250.0)
- added L3: L 0H, YJYCOIN_YNR8040_6R8M:IND-SMD_L8.0-W8.0, F.Cu at (60.0, -10.0)
- added R10: 450000Ω, FOJAN_FRC0402F4503TS:R0402, F.Cu at (60.0, -110.0)
- added R11: 240000Ω, FOJAN_FRC0402F2403TS:R0402, F.Cu at (60.0, -220.0)
- added R12: 53600Ω, UNI_ROYAL_0402WGF5362TCE:R0402, F.Cu at (60.0, -30.0)
- added R13: 10200Ω, UNI_ROYAL_0402WGF1022TCE:R0402, F.Cu at (60.0, 0.00)
- added R14: 16900Ω, UNI_ROYAL_0402WGF1692TCE:R0402, F.Cu at (60.0, -210.0)
- added R15: 91000Ω, YAGEO_RC0402FR_0791KL:R0402, F.Cu at (60.0, -80.0)
- added R16: 450000Ω, FOJAN_FRC0402F4503TS:R0402, F.Cu at (60.0, -190.0)
- added R17: 240000Ω, FOJAN_FRC0402F2403TS:R0402, F.Cu at (60.0, -290.0)
- added R18: 53600Ω, UNI_ROYAL_0402WGF5362TCE:R0402, F.Cu at (60.0, -70.0)
- added R19: 1Ω, UNI_ROYAL_1210W2F100KT5E:R1210, F.Cu at (0.00, 0.00)
- added R20: 1Ω, UNI_ROYAL_1210W2F100KT5E:R1210, F.Cu at (0.00, -10.0)
- added R21: 1Ω, UNI_ROYAL_1210W2F100KT5E:R1210, F.Cu at (0.00, -20.0)
- added R8: 16900Ω, UNI_ROYAL_0402WGF1692TCE:R0402, F.Cu at (60.0, -120.0)
- added R9: 91000Ω, YAGEO_RC0402FR_0791KL:R0402, F.Cu at (60.0, -40.0)
- added U2: , Texas_Instruments_TPS54560DDAR:SOIC-8_L5.0-W4.0-P1.27-LS6.0-BL-EP2.0, F.Cu at (20.0, 0.00)
- added U3: , Texas_Instruments_TPS54560DDAR:SOIC-8_L5.0-W4.0-P1.27-LS6.0-BL-EP2.0, F.Cu at (40.0, 0.00)
- R5: value 1Ω -> 240000Ω; footprint UNI_ROYAL_1210W2F100KT5E:R1210 -> FOJAN_FRC0402F2403TS:R0402
- R6: value 243000Ω -> 53600Ω; footprint UNI_ROYAL_0402WGF2433TCE:R0402 -> UNI_ROYAL_0402WGF5362TCE:R0402
- R7: value 53600Ω -> 10200Ω; footprint UNI_ROYAL_0402WGF5362TCE:R0402 -> UNI_ROYAL_0402WGF1022TCE:R0402
- moved R3 306.0 mm to (60.0, -320.0)
- moved R6 292.6 mm to (60.0, -310.0)
- moved R7 257.6 mm to (60.0, -240.0)
- moved R2 232.6 mm to (60.0, -60.0)
- moved C2 230.2 mm to (60.0, -200.0)
- moved C1 229.8 mm to (60.0, -100.0)
- moved C3 229.8 mm to (60.0, -90.0)
- moved R4 229.8 mm to (60.0, -50.0)
- moved R1 224.1 mm to (60.0, -150.0)
- moved R5 222.3 mm to (60.0, -130.0)
- moved C4 214.2 mm to (60.0, -140.0)
- moved D1 203.9 mm to (10.0, 0.00)
- moved L1 173.1 mm to (60.0, -160.0), turned to 0 degrees
- turned U1 to 0 degrees
Connections:
- net power_in-hv renamed dut12-power_in-hv
- L1 pad 2: power_out-hv -> dut12-power_out-hv
- R5 pad 1: power_out-hv -> RT_CLK
- R6 pad 1: RT_CLK -> dut12-power_out-hv
- R6 pad 2: anode -> FB
- R7 pad 1: power_out-hv -> dut24-FB
- R7 pad 2: FB -> dut24-power_out-anode
Routing:
- net EN: track 26.8 -> 0.00 mm, vias 21 -> 0
- net 0: track 22.4 -> 0.00 mm, vias 7 -> 0
- net dut12-power_in-hv: track 17.5 -> 0.00 mm
- net power_out-hv: track 12.4 -> 0.00 mm, vias 7 -> 0
- net FB: track 9.00 -> 0.00 mm
- removed copper zone on F.Cu, net 0
- removed copper zone on F.Cu, net EN
- removed copper zone on F.Cu, net dut12-power_in-hv
- removed copper zone on F.Cu, net power_out-hv

Commit message: Requirements working, slightly editable
Parts:
- removed C10, C6: 0F, Samsung_Electro_Mechanics_CL10C470JB8NNNC:C0603
- removed C11, C7: 0F, FH_0805B472K500NT:C0805
- removed C12, C8: 0F, Samsung_Electro_Mechanics_CL21A106KAYNNNE:C0805
- removed C5, C9: 0F, YAGEO_CC0603KRX7R9BB104:C0603
- removed D2, D3: , STMicroelectronics_STPS340U:SMB_L4.6-W3.6-LS5.3-RD
- removed L2, L3: L 0H, YJYCOIN_YNR8040_6R8M:IND-SMD_L8.0-W8.0
- removed R10, R16: 450000Ω, FOJAN_FRC0402F4503TS:R0402
- removed R11, R17: 240000Ω, FOJAN_FRC0402F2403TS:R0402
- removed R12, R18: 53600Ω, UNI_ROYAL_0402WGF5362TCE:R0402
- removed R13: 10200Ω, UNI_ROYAL_0402WGF1022TCE:R0402
- removed R14, R8: 16900Ω, UNI_ROYAL_0402WGF1692TCE:R0402
- removed R15, R9: 91000Ω, YAGEO_RC0402FR_0791KL:R0402
- removed R19, R20, R21: 1Ω, UNI_ROYAL_1210W2F100KT5E:R1210
- removed U2, U3: , Texas_Instruments_TPS54560DDAR:SOIC-8_L5.0-W4.0-P1.27-LS6.0-BL-EP2.0
- R5: value 240000Ω -> 1Ω; footprint FOJAN_FRC0402F2403TS:R0402 -> UNI_ROYAL_1210W2F100KT5E:R1210
- R6: value 53600Ω -> 240000Ω; footprint UNI_ROYAL_0402WGF5362TCE:R0402 -> FOJAN_FRC0402F2403TS:R0402
- R7: value 10200Ω -> 53600Ω; footprint UNI_ROYAL_0402WGF1022TCE:R0402 -> UNI_ROYAL_0402WGF5362TCE:R0402
- moved R3 300.7 mm to (80.0, -20.0)
- moved R7 191.0 mm to (80.0, -430.0)
- moved R6 121.7 mm to (80.0, -190.0)
- moved C2 111.8 mm to (80.0, -310.0)
- moved R1 92.2 mm to (80.0, -240.0)
- moved L1 72.8 mm to (80.0, -230.0)
- moved C4 63.2 mm to (80.0, -200.0)
- moved R4 63.2 mm to (80.0, -110.0)
- moved C1 53.9 mm to (80.0, -150.0)
- moved C3 53.9 mm to (80.0, -140.0)
- moved R2 36.1 mm to (80.0, -90.0)
- moved R5 36.1 mm to (80.0, -100.0)
Connections:
- net dut12-power_in-hv renamed power_in-hv
- L1 pad 2: dut12-power_out-hv -> power_out-hv
- R5 pad 1: RT_CLK -> power_out-hv
- R6 pad 1: dut12-power_out-hv -> RT_CLK
- R6 pad 2: FB -> anode
- R7 pad 1: dut24-FB -> power_out-hv
- R7 pad 2: dut24-power_out-anode -> FB
