File: examples/buck_converter/layouts/default/default.kicad_pcb (KiCad board)
At the start: 2 copper layers, 14 parts

Commit message: checkin work
Parts:
- R6: value 1000Ω -> 10000Ω; footprint UNI_ROYAL_1210W2J0102T5E:R1210 -> YAGEO_RC1210FR_0710KL:R1210
Changed lines of the file:
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@@
 		)
 	)
-	(footprint "UNI_ROYAL_1210W2J0102T5E:R1210"
+	(footprint "YAGEO_RC1210FR_0710KL:R1210"
 		(layer "F.Cu")
 		(at 0 -10 0)
@@
 			)
 		)
-		(property "Value" "1000Ω"
+		(property "Value" "10000Ω"
 			(at 0 4)
 			(layer "F.Fab")
@@
 			)
 		)
-		(property "LCSC" "C270888"
+		(property "LCSC" "C309586"
 			(at 0 0 0)
 			(layer "User.9")
 			(hide yes)
 		)
-		(property "Manufacturer" "UNI-ROYAL(Uniroyal Elec)"
+		(property "Manufacturer" "YAGEO"
 			(at 0 0 0)
 			(layer "User.9")
@@
 			(hide yes)
 		)
-		(property "PARAM_resistance" "{\"type\": \"Quantity_Interval_Disjoint\", \"data\": {\"intervals\": {\"type\": \"Numeric_Interval_Disjoint\", \"data\": {\"intervals\": [{\"type\": \"Numeric_Interval\", \"data\": {\"min\": 949.9999992549419, \"max\": 1050.000000745058}}]}}, \"unit\": \"ohm\"}}"
+		(property "PARAM_resistance" "{\"type\": \"Quantity_Interval_Disjoint\", \"data\": {\"intervals\": {\"type\": \"Numeric_Interval_Disjoint\", \"data\": {\"intervals\": [{\"type\": \"Numeric_Interval\", \"data\": {\"min\": 9900.000002235174, \"max\": 10099.999997764826}}]}}, \"unit\": \"ohm\"}}"
 			(at 0 0 0)
 			(layer "User.9")
 			(hide yes)
 		)
-		(property "Partnumber" "1210W2J0102T5E"
+		(property "Partnumber" "RC1210FR-0710KL"
 			(at 0 0 0)
 			(layer "User.9")
 			(hide yes)
 		)
-		(property "Datasheet" "https://www.lcsc.com/datasheet/lcsc_datasheet_2205312300_UNI-ROYAL-Uniroyal-Elec-1210W2J0102T5E_C270888.pdf"
+		(property "Datasheet" "https://wmsc.lcsc.com/wmsc/upload/file/pdf/v2/lcsc/2304140030_YAGEO-RC1210FR-0710KL_C309586.pdf"
 			(at 0 0 0)
 			(layer "User.9")
 			(hide yes)
 		)
-		(property "resistance" "1000±5.0%Ω"
+		(property "resistance" "10000±1.0%Ω"
 			(at 0 0 0)
 			(layer "User.9")
@@
 			(hide yes)
 		)
-		(property "lcsc_id" "C270888"
+		(property "lcsc_id" "C309586"
 			(at 0 0 0)
 			(layer "User.9")
@@
 		)
 		(embedded_fonts no)
-		(model "${KIPRJMOD}/../../parts/UNI_ROYAL_1210W2J0102T5E/R1210_L3.2-W2.6-H0.6.step"
+		(model "${KIPRJMOD}/../../parts/YAGEO_RC1210FR_0710KL/R1210_L3.2-W2.6-H0.6.step"
 			(offset
 				(xyz 0 0 -0)
