File: examples/buck_converter/layouts/model-validation/model-validation.kicad_pcb (KiCad board)
At the start: 2 copper layers, 0 parts

Commit message: checkin work
Parts:
- added C1: 0F, YAGEO_CC0603KRX7R9BB104:C0603, F.Cu at (-162.0, -159.4)
- added C2: 0F, Samsung_Electro_Mechanics_CL10C470JB8NNNC:C0603, F.Cu at (-162.0, -139.4)
- added C3: 0F, FH_0805B472K500NT:C0805, F.Cu at (-162.0, -149.4)
- added C4: 0F, Samsung_Electro_Mechanics_CL21A106KAYNNNE:C0805, F.Cu at (-152.0, -109.4)
- added C5: 0F, YAGEO_CC0603KRX7R9BB104:C0603, F.Cu at (0.00, -10.0)
- added C6: 0F, YAGEO_CC0603KRX7R9BB104:C0603, F.Cu at (0.00, 0.00)
- added C7: 0F, YAGEO_CC0603KRX7R9BB104:C0603, F.Cu at (0.00, -30.0)
- added C8: 0F, YAGEO_CC0603KRX7R9BB104:C0603, F.Cu at (0.00, -20.0)
- added D1: , STMicroelectronics_STPS340U:SMB_L4.6-W3.6-LS5.3-RD, F.Cu at (-162.0, -109.4)
- added L1: L 0H, YJYCOIN_YNR8040_6R8M:IND-SMD_L8.0-W8.0, F.Cu at (-8.08, -0.80)
- added R1: 10200Ω, UNI_ROYAL_0402WGF1022TCE:R0402, F.Cu at (-162.0, -109.4)
- added R2: 16900Ω, UNI_ROYAL_0402WGF1692TCE:R0402, F.Cu at (-162.0, -129.4)
- added R3: 91000Ω, YAGEO_RC0402FR_0791KL:R0402, F.Cu at (-162.0, -109.4)
- added R4: 450000Ω, FOJAN_FRC0402F4503TS:R0402, F.Cu at (-162.0, -109.4)
- added R5: 10000Ω, YAGEO_RC1210FR_0710KL:R1210, F.Cu at (-162.0, -119.4)
- added R6: 240000Ω, FOJAN_FRC0402F2403TS:R0402, F.Cu at (-162.0, -119.4)
- added R7: 53600Ω, UNI_ROYAL_0402WGF5362TCE:R0402, F.Cu at (-162.0, -119.4)
- added U1: , Texas_Instruments_TPS54560DDAR:SOIC-8_L5.0-W4.0-P1.27-LS6.0-BL-EP2.0, F.Cu at (0.00, 0.00)
Routing:
- net 0: track 0.00 -> 43.8 mm, vias 0 -> 14
- net EN: track 0.00 -> 26.8 mm, vias 0 -> 21
- net power_in-hv: track 0.00 -> 17.5 mm
- added copper zone on F.Cu, net 0
- added copper zone on F.Cu, net EN
- added copper zone on F.Cu, net power_in-hv
